File: CTS-SAT-2 CSS in-house/CTS-SAT-2 CSS in-house.kicad_sch (KiCad schematic)
At the start: 56 parts, among them J1 Conn_01x05_Socket, J12 Socket_1x2, J13 Socket_1x2, J18 Socket_1x2, J19 Socket_1x2, U1 POPA4383PWR, U2 POPA4383PWR, U3 ADS7128IRTET

Commit message: Managing signal integrity
Add ground pours, stitching vias, still need alot to fix.
Parts:
- C19, C20, C9: footprint Capacitor_SMD:C_0402_1005Metric_Pad0.74x0.62mm_HandSolder -> Capacitor_SMD:C_0603_1608Metric_Pad1.08x0.95mm_HandSolder
- J1: footprint Connector_PinHeader_2.54mm:PinHeader_1x05_P2.54mm_Vertical -> Connector_PinHeader_2.54mm:PinHeader_1x05_P2.54mm_Vertical_SMD_Pin1Left
- R20, R23: footprint Resistor_SMD:R_0201_0603Metric_Pad0.64x0.40mm_HandSolder -> Resistor_SMD:R_0402_1005Metric_Pad0.72x0.64mm_HandSolder
Changed lines of the file:
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@@
 			)
 		)
-		(property "Footprint" "Capacitor_SMD:C_0402_1005Metric_Pad0.74x0.62mm_HandSolder"
+		(property "Footprint" "Capacitor_SMD:C_0603_1608Metric_Pad1.08x0.95mm_HandSolder"
 			(at 330.2 72.6948 0)
 			(hide yes)
@@
 			)
 		)
-		(property "Footprint" "Resistor_SMD:R_0201_0603Metric_Pad0.64x0.40mm_HandSolder"
+		(property "Footprint" "Resistor_SMD:R_0402_1005Metric_Pad0.72x0.64mm_HandSolder"
 			(at 342.9 100.838 90)
 			(hide yes)
@@
 			)
 		)
-		(property "Footprint" "Capacitor_SMD:C_0402_1005Metric_Pad0.74x0.62mm_HandSolder"
+		(property "Footprint" "Capacitor_SMD:C_0603_1608Metric_Pad1.08x0.95mm_HandSolder"
 			(at 390.1948 68.58 0)
 			(hide yes)
@@
 			)
 		)
-		(property "Footprint" "Connector_PinHeader_2.54mm:PinHeader_1x05_P2.54mm_Vertical"
+		(property "Footprint" "Connector_PinHeader_2.54mm:PinHeader_1x05_P2.54mm_Vertical_SMD_Pin1Left"
 			(at 358.14 120.65 0)
 			(hide yes)
@@
 			)
 		)
-		(property "Footprint" "Resistor_SMD:R_0201_0603Metric_Pad0.64x0.40mm_HandSolder"
+		(property "Footprint" "Resistor_SMD:R_0402_1005Metric_Pad0.72x0.64mm_HandSolder"
 			(at 332.74 100.838 90)
 			(hide yes)
@@
 			)
 		)
-		(property "Footprint" "Capacitor_SMD:C_0402_1005Metric_Pad0.74x0.62mm_HandSolder"
+		(property "Footprint" "Capacitor_SMD:C_0603_1608Metric_Pad1.08x0.95mm_HandSolder"
 			(at 340.36 82.2452 0)
 			(hide yes)

Commit message: Small edits to schematic
Changed some photodiode errors
Connections:
- net 3V3_SUPPLY_1: now also LED1.2 (CATHODE), LED2.2 (CATHODE), LED3.2 (CATHODE), LED4.2 (CATHODE), LED5.2 (CATHODE), LED6.2 (CATHODE), LED7.2 (CATHODE), LED8.2 (CATHODE)
- net GND: no longer LED1.2 (CATHODE), LED2.2 (CATHODE), LED3.2 (CATHODE), LED4.2 (CATHODE), LED5.2 (CATHODE), LED6.2 (CATHODE), LED7.2 (CATHODE), LED8.2 (CATHODE)

Commit message: Final schematic
Schematic is fully finished
Parts:
- added C17: 100 uF, Capacitor_SMD:C_0603_1608Metric_Pad1.08x0.95mm_HandSolder, symbol Device:C
- added C18: 22 uF, Capacitor_SMD:C_0603_1608Metric_Pad1.08x0.95mm_HandSolder, symbol Device:C
- added C23, C24, C27: 100 nF, Capacitor_SMD:C_0603_1608Metric_Pad1.08x0.95mm_HandSolder, symbol Device:C
- added C25, C26: 10 uF, Capacitor_SMD:C_0603_1608Metric_Pad1.08x0.95mm_HandSolder, symbol Device:C
- added R17, R18: 10 Ω, Capacitor_SMD:C_0603_1608Metric_Pad1.08x0.95mm_HandSolder, symbol Device:R
- C10, C11, C12, C2, C3, C4, C5, C6: value 32 nF -> 33 nF
- R2, R3, R4, R5, R6, R7, R8, R9: value 1.01 MΩ -> 3.3 kΩ; footprint Resistor_SMD:R_0805_2012Metric_Pad1.20x1.40mm_HandSolder -> Resistor_SMD:R_0603_1608Metric_Pad0.98x0.95mm_HandSolder
- R20, R23: footprint Resistor_SMD:R_0402_1005Metric_Pad0.72x0.64mm_HandSolder -> Resistor_SMD:R_0603_1608Metric_Pad0.98x0.95mm_HandSolder
Connections:
- net 1.65V_VGND_1: now also C17.1
- net 3V3_SUPPLY_1: now also C18.1, C23.1, R17.2, R18.2; no longer C21.2, C22.2, LED1.2 (CATHODE), LED2.2 (CATHODE), LED3.2 (CATHODE), LED4.2 (CATHODE), LED5.2 (CATHODE), LED6.2 (CATHODE), LED7.2 (CATHODE), LED8.2 (CATHODE)
- net ARRAY_SIGNAL_1: no longer LED2.1 (ANODE)
- net ARRAY_SIGNAL_4: no longer LED5.1 (ANODE)
- net GND: now also C17.2, C18.2, C23.2, C24.2, C25.1, C26.1, C27.2
- new net: C26.2, C27.1, LED1.2 (CATHODE), R18.1
- new net 3V3_U1: C21.2, C22.2, C24.1, C25.2, LED2.2 (CATHODE), LED3.2 (CATHODE), LED4.2 (CATHODE), LED5.2 (CATHODE), LED6.2 (CATHODE), LED7.2 (CATHODE), LED8.2 (CATHODE), R17.1

Commit message: Pcb designing
Connections:
- net ARRAY_SIGNAL_1: now also LED2.1 (ANODE)
- net ARRAY_SIGNAL_4: now also LED5.1 (ANODE)
Changed lines of the file:
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@@
-	(wire
-		(pts
-			(xy 64.77 162.56) (xy 63.5 162.56)
-		)
-		(stroke
-			(width 0)
-			(type default)
-		)
-	)
 	(wire
 		(pts
@@
 	)
 	(label "ARRAY_SIGNAL_1"
-		(at 63.5 162.56 0)
+		(at 62.23 162.56 0)
 		(effects
 			(font
@@
 	)
 	(label "ARRAY_SIGNAL_4"
-		(at 63.5 215.9 0)
-		(effects
-			(font
+		(at 62.23 215.9 0)
+		(effects
+			(font

Commit message: Final before design review
Fully finished schematic, pcb placement and pcb routing.
Connections:
- net 3V3_U1: now also C21.1, C22.1, U1.4 (V+), U2.4 (V+); no longer C21.2, C22.2
- net GND: now also C21.2, C22.2
- net CSS_ARRAY_SIGNAL: now reaches C4.1, J13.2 (Pin_2), LED1.1 (ANODE), R4.1, U1.13 (-IN_D)
Other:
- note added: "RC filter"
- moved on the sheet: C21, C22
